File: M2.kicad_sch (KiCad schematic)
At the start: 4 parts, among them J13 Bus_M.2_Socket_M

Commit message: add impedance spec in the datasheet
Parts:
- C100: footprint (none) -> Capacitor_SMD:C_1206_3216Metric
Changed lines of the file:
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@@
 			)
 		)
-		(property "Footprint" ""
+		(property "Footprint" "Capacitor_SMD:C_1206_3216Metric"
 			(at 109.5248 26.67 0)
 			(effects
