File: MAINPAGE.kicad_sch (KiCad schematic)
At the start: 17 parts, among them J1 USB_C_Receptacle

Commit message: add impedance spec in the datasheet
Parts:
- added C103: 100n, Capacitor_SMD:C_0402_1005Metric, symbol Device:C
- added J10: Programming Headder, Connector_PinHeader_2.54mm:PinHeader_1x07_P2.54mm_Vertical, symbol Connector_Generic:Conn_01x07
- added R139, R140, R141: 5K1, symbol Device:R_US
- added R152, R153: 33R, Resistor_SMD:R_0402_1005Metric, symbol Device:R_US
- added U10: W25X20CLSNIG, Package_SO:SOIC-8_3.9x4.9mm_P1.27mm, symbol Memory_Flash:W25X20CLSN
- FID1, FID2, FID3: footprint (none) -> Fiducial:Fiducial_0.75mm_Mask1.5mm
- R111: footprint (none) -> Resistor_SMD:R_0402_1005Metric; now not fitted; now left out of the parts list
Connections:
- net GND: now also C103.1, J10.7 (Pin_7), U10.4 (GND)
- new net: R140.2, U10.7 (~{HOLD})
- new net: R139.2, U10.3 (~{WP})
- new net +2V5: C103.2, J10.1 (Pin_1), R139.1, R140.1, R141.1, U10.8 (VCC)
- new net PI_RX: R152.2
- new net PI_TX: R153.2
- new net SWITCH_RESET: J10.6 (Pin_6)
- new net SWITCH_RX: R153.1
- new net SWITCH_TX: R152.1
- new net VSC_SI_CLK: J10.3 (Pin_3), U10.6 (CLK)
- new net VSC_SI_DI: J10.4 (Pin_4), U10.5 (DI/IO_{0})
- new net VSC_SI_DO: J10.5 (Pin_5), U10.2 (DO/IO_{1})
- new net VSC_SI_~{CS0}: J10.2 (Pin_2), R141.2, U10.1 (~{CS})
- no-connect marks 12 -> 10
Other:
- sheet SWITCH ports: added GPIO4, VSC_SI_CLK, VSC_SI_DI, VSC_SI_DO, VSC_SI_~{CS0}, ~{PME_N}/GPIO6; removed SI_CLK, SI_DI, SI_DO, SI_~{CS0}
- note added: "SPI0"
- note added: "SPI1"
