File: SWITCH.kicad_sch (KiCad schematic)
At the start: 186 parts, among them J10 Conn_01x03, J11 Conn_01x03, J12 Conn_01x03, J2 Conn_01x03, J3 SFP+, J4 SFP+, J5 Conn_01x07, J6 12401610E4-2A, J9 Conn_01x07, U2 74HC164, U3 VSC7512XMY, U4 KSZ9477STXI, U5 LAN7801T/9JX, U7 PI3USB302-AZBEX, U8 LMV331IDBVR, U9 93LC66A/SN, X1 SG-8018CG 125.000000MHz TJHPA, X2 SG-8018CG 125.000000MHz TJHPA, Y1 ASDMB-25.000MHZ-LC-T, Y2 ASDMB-25.000MHZ-LC-T

Commit message: add impedance spec in the datasheet
Parts:
- removed D47, D48, D49, D50, D51, D52, D53, D54, D55, D56, D58, D59, D60, D61, D62, D63, D64, D65: LED_Dual_Bidirectional, symbol Device:LED_Dual_Bidirectional
- removed J10, J11, J12, J2: Conn_01x03, symbol Connector_Generic:Conn_01x03
- added C102, C105, C106, C107, C108, C109, C110, C111, C112, C113, C114, C119, C120: 100n, Capacitor_SMD:C_0402_1005Metric, symbol Device:C
- added C104, C117: 10u, Capacitor_SMD:C_1206_3216Metric, symbol Device:C
- added C115, C116: 1u, Capacitor_SMD:C_0603_1608Metric, symbol Device:C
- added C118: 4u7, Capacitor_SMD:C_1206_3216Metric, symbol Device:C
- added D37, D39, D40, D41, D42, D43, D44, D45, D46, D47, D48, D49, D50, D51, D52, D53, D54, D55: LED, symbol Device:LED
- added D38: 1N4148W, Diode_SMD:D_SOD-123, symbol Diode:1N4148W
- added R135, R136, R137, R138: 0R, symbol Device:R_US
- added R142: 5K1, symbol Device:R_US
- added R143, R144, R145: 750R, symbol Device:R_US
- added R146: 6K04, symbol Device:R_US
- added R147: 0R, Resistor_SMD:R_0402_1005Metric, symbol Device:R_US
- added R148, R149, R150, R151: 5K1, Resistor_SMD:R_0805_2012Metric, symbol Device:R_US
- C65, C66, C81, C82, C92: footprint (none) -> Capacitor_SMD:C_1206_3216Metric
- D57: value LED_Dual_Bidirectional -> XZMYKVG55W-4; footprint (none) -> LED_SMD:LED_1206_3216Metric
- J5, J9: footprint (none) -> Connector_PinHeader_2.54mm:PinHeader_1x07_P2.54mm_Vertical
- R113, R37, R75, R76, R77, R78, R79, R80, R81, R82, R83, R84: value 4K7 -> 5K1
- R123, R125, R45, R46, R49, R50, R55, R56: value 4K7 -> 5K1; footprint (none) -> Resistor_SMD:R_0805_2012Metric
- R124, R126: value 4K7 -> 5K1; footprint (none) -> Resistor_SMD:R_0805_2012Metric; now not fitted; now left out of the parts list
- R127, R133, R40, R41, R42, R44, R69, R70, R71, R72, R73, R74, R85, R86, R87, R88, R89, R90, R91: footprint (none) -> Resistor_SMD:R_0402_1005Metric
- RJ1: value ~ -> DS1130-S80BP
Connections:
- net +1V0: now also C102.2, C116.2, C118.1, C119.2, C120.2, D37.2 (A), D39.2 (A), D40.2 (A), D41.2 (A), D42.2 (A), D43.2 (A), D44.2 (A), D45.2 (A), D46.2 (A), D47.2 (A), D48.2 (A), D49.2 (A), D50.2 (A), D51.2 (A), D52.2 (A), D53.2 (A), D54.2 (A), D55.2 (A)
- net +1V2_USB: now also C105.2, C106.2, C114.2, C115.2, C117.1, R147.1; no longer C92.1, L1.1, U5.22 (VDD12_SW_FB)
- net +2V5: now also R123.1, R125.1, C107.2, C108.2, C109.2, C110.2, C111.2, C112.2, C113.2, D38.1 (K), R142.1, R146.1, R148.1, R150.1
- net GND: now also R124.2, R126.2, C102.1, C104.2, C105.1, C106.1, C107.1, C108.1, C109.1, C110.1, C111.1, C112.1, C113.1, C114.1, C115.1, C116.1, C117.2, C118.2, C119.1, C120.1, R143.2, R144.2, R145.2, R149.2, R151.2
- net LED0_0_K: now also D48.1 (K)
- net LED0_1_K: now also D49.1 (K)
- net LED1_0: now also D37.1 (K)
- net LED1_0_K: now also D50.1 (K)
- net LED1_1: now also D39.1 (K)
- net LED1_1_K: now also D51.1 (K)
- net LED2_0: now also D40.1 (K)
- net LED2_0_K: now also D52.1 (K)
- net LED2_1: now also D41.1 (K)
- net LED2_1_K: now also D53.1 (K)
- net LED3_0: now also D42.1 (K)
- net LED3_0_K: now also D54.1 (K)
- net LED3_1: now also D43.1 (K)
- net LED3_1_K: now also D55.1 (K)
- net LED4_0: now also D44.1 (K)
- net LED4_1: now also D45.1 (K)
- net LED5_0: now also D46.1 (K)
- net LED5_1: now also D47.1 (K)
- net SFP1_RATESEL: now also R124.1
- net SFP1_SCL: now also R148.2, R149.1; no longer R125.2
- net SFP2_RATESEL: now also R125.2, R126.1; no longer R124.2
- net SFP2_SCL: now also R150.2, R151.1; no longer R126.2
- net ~{RESET}: now also C104.1, D38.2 (A), R142.2
- net RXD6_2: now reaches R72.1
- net RXD6_2: now also U4.63 (RXD6_2); no longer U4.53 (TXD6_2)
- net RXD2: now reaches R72.2, U5.16 (RXD2)
- net at R97.2, U4.105 (LED1_0): now also R143.1
- net at R98.2, U4.106 (LED1_1): now also R144.1
- net at R100.2, U4.92 (LED2_1): now also R145.1
- net at U4.95 (SYNCLKO): now also R146.2
- net RXD6_0: now reaches R70.1
- net RXD6_0: now also U4.65 (RXD6_0); no longer U4.55 (TXD6_0)
- net RXD0: now reaches R70.2, U5.14 (RXD0)
- net RX_CLK6/REFCLKO6: now reaches R74.1
- net RX_CLK6/REFCLKO6: now also U4.57 (RX_CLK6/REFCLKO6); no longer U4.48 (TX_CLK6/REFCLKI6)
- net RXC: now reaches R74.2, U5.12 (RXC)
- net VSC_125MHz: now reaches R38.2, R39.1, U3.84 (REFCLK_P)
- net VBUS_USB_ETH_PHY: now reaches C93.2, J6.A4 (VBUS), J6.A9 (VBUS), J6.B4 (VBUS), J6.B9 (VBUS), R120.1, R121.2
- net at J6.A5 (CC1), R96.1: now also R135.2, R137.2; no longer U8.3 (-)
- net at J6.B5 (CC2), R68.1: now also R136.2, R138.2; no longer U8.1 (+)
- net LAN_125MHz: now reaches R114.2, U5.19 (CLK125)
- net RX_CTL6: now reaches R69.1
- net RX_CTL6: now also U4.58 (RX_DV6/CRS_DV6/RX_CTL6); no longer U4.49 (TX_EN6/TX_CTL6)
- net RX_CTL: now reaches R69.2, U5.13 (RX_CTL)
- net RXD6_3: now reaches R73.1
- net RXD6_3: now also U4.62 (RXD6_3); no longer U4.52 (TXD6_3)
- net RXD6_1: now reaches R71.1
- net RXD6_1: now also U4.64 (RXD6_1); no longer U4.54 (TXD6_1)
- net TX_CLK6/REFCLKI6: now reaches R85.2
- net TX_CLK6/REFCLKI6: now also U4.48 (TX_CLK6/REFCLKI6); no longer U4.57 (RX_CLK6/REFCLKO6)
- net TX_CTL6: now reaches R90.2
- net TX_CTL6: now also U4.49 (TX_EN6/TX_CTL6); no longer U4.58 (RX_DV6/CRS_DV6/RX_CTL6)
- net TXD6_3: now reaches R89.2
- net TXD6_3: now also U4.52 (TXD6_3); no longer U4.62 (RXD6_3)
- net TXD6_2: now reaches R88.2
- net TXD6_2: now also U4.53 (TXD6_2); no longer U4.63 (RXD6_2)
- net TXD6_1: now reaches R87.2
- net TXD6_1: now also U4.54 (TXD6_1); no longer U4.64 (RXD6_1)
- net TXD6_0: now reaches R86.2
- net TXD6_0: now also U4.55 (TXD6_0); no longer U4.65 (RXD6_0)
- net TXD3: now reaches R89.1, U5.4 (TXD3)
- net TXD0: now reaches R86.1, U5.8 (TXD0)
- net RXD3: now reaches R73.2, U5.17 (RXD3)
- net TXC: now reaches R85.1, U5.10 (TXC)
- net TX_CTL: now reaches R90.1, U5.9 (TX_CTL)
- net TXD1: now reaches R87.1, U5.6 (TXD1)
- net RXD1: now reaches R71.2, U5.15 (RXD1)
- net ~{PME_N}/GPIO6: now reaches U5.45 (~{PME_N}/GPIO6)
- net TXD2: now reaches R88.1, U5.5 (TXD2)
- net SI_CLK renamed VSC_SI_CLK
- net SI_DI renamed VSC_SI_DI
- net SI_DO renamed VSC_SI_DO
- net SI_~{CS0} renamed VSC_SI_~{CS0}
- new net: C92.1, L1.1, R147.2, U5.22 (VDD12_SW_FB)
- new net: R135.1, R138.1, U8.3 (-)
- new net: R136.1, R137.1, U8.1 (+)
- no-connect marks 25 -> 24
Other:
- moved on the sheet: C83, C89, C90, C91, C92, C93, C94, C95, C96, C97, C98, D57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
